Commit message: Task1 Re-evaluating

File: my_rb1_description/urdf/my_rb1_robot.urdf (robot description, URDF)
Before this commit: robot robot, 7 links, 6 joints
Links:
- link link_chassis: mass 10 -> 19.5
Joints:
- joint joint_chassis_back_caster_wheel: type continuous -> fixed
- joint joint_chassis_base_link: type continuous -> fixed
- joint joint_chassis_front_caster_wheel: type continuous -> fixed

Commit message: task1 re-evaluating.. Kannan informally approved

File: my_rb1_description/urdf/my_rb1_robot.urdf (robot description, URDF)
Before this commit: robot robot, 7 links, 6 joints
Joints:
- joint joint_chassis_base_link: origin xyz=0 0 -0.15 rpy=0 0 0 -> xyz=0 0 0 rpy=0 0 0

Commit message: switch wheels name from left to right, and caster wheels name from front to back

File: my_rb1_description/urdf/my_rb1_robot.urdf (robot description, URDF)
Before this commit: robot robot, 7 links, 6 joints
Links:
- added link link_base_footprint, mass 1; collision box size=0 0 0; visual box size=0 0 0
Joints:
- added joint joint_chassis_base_footprint: type fixed, parent link_chassis, child link_base_footprint, origin xyz=0 0 -0.15 rpy=0 0 0, axis 0 1 0, limit effort=10000 velocity=1000
- joint joint_chassis_back_caster_wheel: origin xyz=0.1 0.0 -0.15 rpy=0 0 0 -> xyz=-0.1 0.0 -0.15 rpy=0 0 0
- joint joint_chassis_front_caster_wheel: origin xyz=-0.1 0.0 -0.15 rpy=0 0 0 -> xyz=0.1 0.0 -0.15 rpy=0 0 0
- joint joint_chassis_left_wheel: origin xyz=0 -0.2 -0.15 rpy=0 0 0 -> xyz=0 0.2 -0.15 rpy=0 0 0
- joint joint_chassis_right_wheel: origin xyz=0 0.2 -0.15 rpy=0 0 0 -> xyz=0 -0.2 -0.15 rpy=0 0 0

Commit message: switch caster wheels name

File: my_rb1_description/urdf/my_rb1_robot.urdf (robot description, URDF)
Before this commit: robot robot, 7 links, 6 joints
Joints:
- joint joint_chassis_back_caster_wheel: origin xyz=0.1 0.0 -0.15 rpy=0 0 0 -> xyz=-0.1 0.0 -0.15 rpy=0 0 0
- joint joint_chassis_front_caster_wheel: origin xyz=-0.1 0.0 -0.15 rpy=0 0 0 -> xyz=0.1 0.0 -0.15 rpy=0 0 0

Commit message: change rotate_service after urdf switch left wheel-right wheel

File: my_rb1_description/urdf/my_rb1_robot.urdf (robot description, URDF)
Before this commit: robot robot, 7 links, 6 joints
Links:
- added link link_base_footprint, mass 1; collision box size=0 0 0; visual box size=0 0 0
Joints:
- added joint joint_chassis_base_footprint: type fixed, parent link_chassis, child link_base_footprint, origin xyz=0 0 -0.15 rpy=0 0 0, axis 0 1 0, limit effort=10000 velocity=1000
- joint joint_chassis_left_wheel: origin xyz=0 -0.2 -0.15 rpy=0 0 0 -> xyz=0 0.2 -0.15 rpy=0 0 0
- joint joint_chassis_right_wheel: origin xyz=0 0.2 -0.15 rpy=0 0 0 -> xyz=0 -0.2 -0.15 rpy=0 0 0

Commit message: change the mass of the robot from 26 to 25

File: my_rb1_description/urdf/my_rb1_robot.urdf (robot description, URDF)
Before this commit: robot robot, 8 links, 7 joints
Links:
- link link_base_footprint: mass 1 -> 0.5
- link link_base_link: mass 1 -> 0.5

Commit message: The wobbling issue solved

File: my_rb1_description/urdf/my_rb1_robot.urdf (robot description, URDF)
Before this commit: robot robot, 8 links, 7 joints
Links:
- link link_back_caster_wheel: mass 1 -> 1.5
- link link_chassis: mass 19.5 -> 10.5
- link link_front_caster_wheel: mass 1 -> 1.5
- link link_left_wheel: mass 1 -> 5
- link link_right_wheel: mass 1 -> 5
